File: hw2/hw2.sch (EAGLE design)
At the start: 0 parts

Commit message: updated schematic
Parts:
- added C1, C2, C3, C4: (no value), hw2:C-US025-025X050
- added C5, C6: (no value), hw2:CPOL-USB45181B
- added J1: USB-MB-H, hw2:USB-MB-H
- added LED1, LED2: (no value), led:LED3MM
- added R1, R2, R3, R4: (no value), hw2:R-US_0207/10
- added U$1: PIC32MX250F128B, hw2:PIC32MX250F128B
- added U$2: SLIDE, hw2:SLIDE
- added U$3: MCP1702, hw2:MCP1702
- added U$4, U$5: PB, hw2:PB
- added U$6, U$7: CONN_08, hw2:CONN_08
- added U$8: PICKIT3, hw2:PICKIT3
- added U$9: OSC, hw2:OSC
